Commit message: update mass, inertia and effort parameters

File: hurba_robot_arm/urdf/robot_arm.urdf (robot description, URDF)
Before this commit: robot robot_arm, 11 links, 10 joints
Links:
- link Fifth: mass 1 -> 2
- link First: mass 1 -> 50
- link Fourth: mass 1 -> 7
- link Gripper_Base: mass 1 -> 0.3
- link Left_Finger: mass 1 -> 0.1
- link Right_Finger: mass 1 -> 0.1
- link Second: mass 1 -> 10
- link Sixth: mass 1 -> 0.5
- link Third: mass 1 -> 10
Joints:
- joint Fourth_joint: limit lower=-3.14 upper=3.14 effort=100.0 velocity=1.0 -> lower=-3.14 upper=3.14 effort=1000.0 velocity=1.0
- joint Third_joint: limit lower=-3.14 upper=3.14 effort=100.0 velocity=1.0 -> lower=-3.14 upper=3.14 effort=3000.0 velocity=1.0

Commit message: fix robot links' inertia

File: hurba_robot_arm/urdf/robot_arm.urdf (robot description, URDF)
Before this commit: robot robot_arm, 11 links, 10 joints
Links:
- link Fifth: mass 2 -> 4.0
- link Left_Finger: mass 0.1 -> 0.05
- link Right_Finger: mass 0.1 -> 0.05
- link Sixth: mass 0.5 -> 1.0
Joints:
- joint Fifth_joint: limit lower=-3.14 upper=3.14 effort=100.0 velocity=1.0 -> lower=-3.14 upper=3.14 effort=400.0 velocity=1.0
- joint First_joint: limit lower=-3.14 upper=3.14 effort=100.0 velocity=1.0 -> lower=-3.14 upper=3.14 effort=5000.0 velocity=1.0
- joint Fourth_joint: limit lower=-3.14 upper=3.14 effort=1000.0 velocity=1.0 -> lower=-3.14 upper=3.14 effort=3000.0 velocity=1.0
- joint Gripper_Base_joint: limit lower=-3.14 upper=3.14 effort=100.0 velocity=1.0 -> lower=-3.14 upper=3.14 effort=200.0 velocity=1.0
- joint Left_Finger_joint: axis 0.0 1 0 -> 0.0 1.0 0.0
- joint Right_Finger_joint: axis 0.0 -1 0 -> 0.0 -1.0 0.0
- joint Sixth_joint: limit lower=-3.14 upper=3.14 effort=100.0 velocity=1.0 -> lower=-3.14 upper=3.14 effort=300.0 velocity=1.0

Commit message: add 3D meshes and camera to the urdf

File: hurba_robot_arm/urdf/robot_arm.urdf (robot description, URDF)
Before this commit: robot robot_arm, 11 links, 10 joints
Links:
- added link camera_link, mass 0.1; collision box size=.05 .05 .05; visual box size=.05 .05 .05
- added link camera_link_optical
- link First: geometry collision cylinder length=0.5 radius=0.4; visual mesh filename=package://hurba_robot_arm/meshes/Link_1.dae
- link Fourth: geometry collision cylinder length=0.5 radius=0.15; visual mesh filename=package://hurba_robot_arm/meshes/Link_4.dae
- link Second: geometry collision cylinder length=0.5 radius=0.3; visual mesh filename=package://hurba_robot_arm/meshes/Link_2.dae
- link Third: geometry collision cylinder length=1.3 radius=0.3; visual mesh filename=package://hurba_robot_arm/meshes/Link_3.dae
Joints:
- added joint camera_joint: type fixed, parent base_link, child camera_link, origin xyz=1.5 0 4.0 rpy=0 1.5707 0, axis 0 1 0
- added joint camera_optical_joint: type fixed, parent camera_link, child camera_link_optical, origin xyz=0 0 0 rpy=-1.5707 0 -1.5707
